File: KNeoPiX_v1.3.kicad_sch (KiCad schematic)
At the start: 32 parts, among them J1 Conn_KNX, J2 Conn_KNX, J3 Screw Terminal - Non Isolated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, J4 Screw Terminal - Isolated IOs, J5 Conn_01x05, J6 Conn_01x05, SW1 Prog BTN, U1 Seeeduino XIAO, U2 LM2937IMP-3.3 / 5.0, U3 ADuM1201AR / ADum1250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

Commit message: New footprint, folder structure
More cleaned UP!
Parts:
- C1, C2, C3, C4, C5, C6, C7: symbol Device:C -> KNeoPix.symbols:C
- D3: symbol Diodes-Incorporated:SMAJ40CA-13-F -> KNeoPix.symbols:SMAJ40CA-13-F
- GN1: symbol OpenKNX_Symbol:OpenKNX_BCU -> KNeoPix.symbols:OpenKNX_BCU
- H1, H2: symbol WAGO-243-131:243-131 -> KNeoPix.symbols:243-131
- J1: symbol OpenKNX_Symbol:Conn_KNX -> KNeoPix.symbols:Conn_KNX
- J2: symbol OpenKNX:Conn_KNX -> KNeoPix.symbols:Conn_KNX
- J3: symbol Connector:Screw_Terminal_01x09 -> KNeoPix.symbols:Screw_Terminal_01x09
- J4: symbol Connector:Screw_Terminal_01x04 -> KNeoPix.symbols:Screw_Terminal_01x04
- J5, J6: symbol Connector_Generic:Conn_01x05 -> KNeoPix.symbols:Conn_01x05
- JP1, JP2, JP3, JP4, JP6: symbol Jumper:SolderJumper_2_Open -> KNeoPix.symbols:SolderJumper_2_Open
- JP5: symbol Jumper:SolderJumper_3_Open -> KNeoPix.symbols:SolderJumper_3_Open
- R1, R2, R3, R4: symbol Device:R_Small -> KNeoPix.symbols:R_Small
- SW1: symbol Switch:SW_Push -> KNeoPix.symbols:SW_Push
- U1: symbol Seeeduino XIAO:SeeeduinoXIAO -> KNeoPix.symbols:SeeeduinoXIAO
- U2: symbol Regulator_Linear:LM2937xMP -> KNeoPix.symbols:LM2937xMP
- U3, U4: symbol Isolator:ADuM1201AR -> KNeoPix.symbols:ADuM1201AR
Changed lines of the file:
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@@
     )
   )
-  (global_label "S_3V3" (shape input) (at 255.27 121.158 180) (fields_autoplaced)
+  (global_label "S_3V3" (shape output) (at 255.27 121.158 180) (fields_autoplaced)
     (effects (font (size 1.27 1.27)) (justify right))
     (property "Intersheetrefs" "${INTERSHEET_REFS}" (at 246.6795 121.158 0)
@@
     )
   )
-  (global_label "S_GND" (shape input) (at 255.016 118.618 180) (fields_autoplaced)
+  (global_label "S_GND" (shape output) (at 255.016 118.618 180) (fields_autoplaced)
     (effects (font (size 1.27 1.27)) (justify right))
     (property "Intersheetrefs" "${INTERSHEET_REFS}" (at 246.0626 118.618 0)
@@
     )
   )
-  (symbol (lib_id "OpenKNX:Conn_KNX") (at 70.866 46.736 180) (unit 1)
+  (symbol (lib_id "KNeoPix.symbols:Conn_KNX") (at 70.866 46.736 180) (unit 1)
     (in_bom yes) (on_board yes) (dnp no)
     (property "Reference" "J2" (at 63.246 45.212 0)
@@
     )
   )
-  (symbol (lib_id "Jumper:SolderJumper_2_Open") (at 383.032 75.946 90) (unit 1)
+  (symbol (lib_id "KNeoPix.symbols:SolderJumper_2_Open") (at 383.032 75.946 90) (unit 1)
     (in_bom yes) (on_board yes) (dnp no)
     (property "Reference" "JP4" (at 383.159 66.421 90)
@@
     )
   )
-  (symbol (lib_id "Device:C") (at 77.978 244.094 0) (unit 1)
+  (symbol (lib_id "KNeoPix.symbols:C") (at 77.978 244.094 0) (unit 1)
     (in_bom yes) (on_board yes) (dnp no)
     (property "Reference" "C4" (at 70.866 242.57 0)
@@
     )
   )
-  (symbol (lib_id "OpenKNX_Symbol:Conn_KNX") (at 84.582 46.736 180) (unit 1)
+  (symbol (lib_id "KNeoPix.symbols:Conn_KNX") (at 84.582 46.736 180) (unit 1)
     (in_bom yes) (on_board yes) (dnp no)
     (property "Reference" "J1" (at 78.232 45.212 0)
@@
     )
   )
-  (symbol (lib_id "Switch:SW_Push") (at 268.478 187.198 90) (unit 1)
+  (symbol (lib_id "KNeoPix.symbols:SW_Push") (at 268.478 187.198 90) (unit 1)
     (in_bom yes) (on_board yes) (dnp no)
     (property "Reference" "SW1" (at 266.446 174.498 90)
@@
     )
   )
-  (symbol (lib_id "WAGO-243-131:243-131") (at 75.946 51.816 180) (unit 1)
+  (symbol (lib_id "KNeoPix.symbols:243-131") (at 75.946 51.816 180) (unit 1)
     (in_bom yes) (on_board yes) (dnp no)
     (property "Reference" "H2" (at 66.04 51.816 0)
@@
     )
   )
-  (symbol (lib_id "Device:C") (at 224.028 56.642 180) (unit 1)
+  (symbol (lib_id "KNeoPix.symbols:C") (at 224.028 56.642 180) (unit 1)
     (in_bom yes) (on_board yes) (dnp no)
     (property "Reference" "C6" (at 224.028 54.102 0)
@@
     )
   )
-  (symbol (lib_id "Device:C") (at 102.87 85.852 0) (unit 1)
+  (symbol (lib_id "KNeoPix.symbols:C") (at 102.87 85.852 0) (unit 1)
     (in_bom yes) (on_board yes) (dnp no)
     (property "Reference" "C5" (at 102.87 83.312 0)
@@
     )
   )
-  (symbol (lib_id "Isolator:ADuM1201AR") (at 196.088 56.642 0) (unit 1)
+  (symbol (lib_id "KNeoPix.symbols:ADuM1201AR") (at 196.088 56.642 0) (unit 1)
     (in_bom yes) (on_board yes) (dnp no) (fields_autoplaced)
     (property "Reference" "U4" (at 196.088 43.434 0)
@@
     )
   )
-  (symbol (lib_id "Jumper:SolderJumper_2_Open") (at 44.704 169.418 90) (unit 1)
+  (symbol (lib_id "KNeoPix.symbols:SolderJumper_2_Open") (at 44.704 169.418 90) (unit 1)
     (in_bom yes) (on_board yes) (dnp no)
     (property "Reference" "JP2" (at 44.704 157.988 90)
@@
     )
   )
-  (symbol (lib_id "Device:R_Small") (at 77.216 102.616 90) (unit 1)
+  (symbol (lib_id "KNeoPix.symbols:R_Small") (at 77.216 102.616 90) (unit 1)
     (in_bom yes) (on_board yes) (dnp no) (fields_autoplaced)
     (property "Reference" "R1" (at 77.216 97.282 90)
@@
     )
   )
-  (symbol (lib_id "OpenKNX_Symbol:OpenKNX_BCU") (at 25.908 45.466 0) (unit 1)
+  (symbol (lib_id "KNeoPix.symbols:OpenKNX_BCU") (at 25.908 45.466 0) (unit 1)
     (in_bom yes) (on_board yes) (dnp no)
     (property "Reference" "GN1" (at 19.558 27.94 0)
@@
     )
   )
-  (symbol (lib_id "Device:R_Small") (at 77.47 69.85 90) (unit 1)
+  (symbol (lib_id "KNeoPix.symbols:R_Small") (at 77.47 69.85 90) (unit 1)
     (in_bom yes) (on_board yes) (dnp no) (fields_autoplaced)
     (property "Reference" "R2" (at 77.47 64.516 90)
@@
     )
   )
-  (symbol (lib_id "Jumper:SolderJumper_2_Open") (at 44.704 140.716 90) (unit 1)
+  (symbol (lib_id "KNeoPix.symbols:SolderJumper_2_Open") (at 44.704 140.716 90) (unit 1)
     (in_bom yes) (on_board yes) (dnp no)
     (property "Reference" "JP1" (at 44.704 128.524 90)
@@
     )
   )
-  (symbol (lib_id "Seeeduino XIAO:SeeeduinoXIAO") (at 312.674 154.686 0) (unit 1)
+  (symbol (lib_id "KNeoPix.symbols:SeeeduinoXIAO") (at 312.674 154.686 0) (unit 1)
     (in_bom yes) (on_board yes) (dnp no)
     (property "Reference" "U1" (at 317.754 147.066 0)
@@
     )
   )
-  (symbol (lib_id "Device:R_Small") (at 195.834 73.406 90) (unit 1)
+  (symbol (lib_id "KNeoPix.symbols:R_Small") (at 195.834 73.406 90) (unit 1)
     (in_bom yes) (on_board yes) (dnp no) (fields_autoplaced)
     (property "Reference" "R4" (at 195.834 67.31 90)
@@
     )
   )
-  (symbol (lib_id "WAGO-243-131:243-131") (at 75.946 39.116 180) (unit 1)
+  (symbol (lib_id "KNeoPix.symbols:243-131") (at 75.946 39.116 180) (unit 1)
     (in_bom yes) (on_board yes) (dnp no)
     (property "Reference" "H1" (at 65.786 39.116 0)
@@
     )
   )
-  (symbol (lib_id "Connector:Screw_Terminal_01x04") (at 270.51 74.93 180) (unit 1)
+  (symbol (lib_id "KNeoPix.symbols:Screw_Terminal_01x04") (at 270.51 74.93 180) (unit 1)
     (in_bom yes) (on_board yes) (dnp no)
     (property "Reference" "J4" (at 270.51 80.518 0)
@@
     )
   )
-  (symbol (lib_id "Connector:Screw_Terminal_01x09") (at 270.51 44.45 180) (unit 1)
+  (symbol (lib_id "KNeoPix.symbols:Screw_Terminal_01x09") (at 270.51 44.45 180) (unit 1)
     (in_bom yes) (on_board yes) (dnp no)
     (property "Reference" "J3" (at 270.51 57.658 0)
@@
     )
   )
-  (symbol (lib_id "Jumper:SolderJumper_3_Open") (at 81.026 168.91 90) (unit 1)
+  (symbol (lib_id "KNeoPix.symbols:SolderJumper_3_Open") (at 81.026 168.91 90) (unit 1)
     (in_bom yes) (on_board yes) (dnp no)
     (property "Reference" "JP5" (at 81.026 157.734 90)
@@
     )
   )
-  (symbol (lib_id "Diodes-Incorporated:SMAJ40CA-13-F") (at 97.282 49.276 90) (unit 1)
+  (symbol (lib_id "KNeoPix.symbols:SMAJ40CA-13-F") (at 97.282 49.276 90) (unit 1)
     (in_bom yes) (on_board yes) (dnp no) (fields_autoplaced)
     (property "Reference" "D3" (at 97.282 42.9259 90)
@@
     )
   )
-  (symbol (lib_id "Connector_Generic:Conn_01x05") (at 263.144 123.698 0) (unit 1)
+  (symbol (lib_id "KNeoPix.symbols:Conn_01x05") (at 263.144 123.698 0) (unit 1)
     (in_bom yes) (on_board yes) (dnp no) (fields_autoplaced)
     (property "Reference" "J5" (at 266.319 123.063 0)
@@
     )
   )
-  (symbol (lib_id "Device:C") (at 44.958 244.094 0) (unit 1)
+  (symbol (lib_id "KNeoPix.symbols:C") (at 44.958 244.094 0) (unit 1)
     (in_bom yes) (on_board yes) (dnp no)
     (property "Reference" "C3" (at 48.26 242.316 0)
@@
     )
   )
-  (symbol (lib_id "Isolator:ADuM1201AR") (at 77.47 85.852 0) (unit 1)
+  (symbol (lib_id "KNeoPix.symbols:ADuM1201AR") (at 77.47 85.852 0) (unit 1)
     (in_bom yes) (on_board yes) (dnp no) (fields_autoplaced)
     (property "Reference" "U3" (at 77.47 73.406 0)
@@
     )
   )
-  (symbol (lib_id "Device:R_Small") (at 195.834 39.878 90) (unit 1)
+  (symbol (lib_id "KNeoPix.symbols:R_Small") (at 195.834 39.878 90) (unit 1)
     (in_bom yes) (on_board yes) (dnp no) (fields_autoplaced)
     (property "Reference" "R3" (at 195.834 34.29 90)
@@
     )
   )
-  (symbol (lib_id "Regulator_Linear:LM2937xMP") (at 60.452 240.284 0) (unit 1)
+  (symbol (lib_id "KNeoPix.symbols:LM2937xMP") (at 60.452 240.284 0) (unit 1)
     (in_bom yes) (on_board yes) (dnp no)
     (property "Reference" "U2" (at 60.452 233.68 0)
@@
     )
   )
-  (symbol (lib_id "Device:C") (at 161.544 56.388 0) (unit 1)
+  (symbol (lib_id "KNeoPix.symbols:C") (at 161.544 56.388 0) (unit 1)
     (in_bom yes) (on_board yes) (dnp no)
     (property "Reference" "C1" (at 159.004 53.848 0)
@@
     )
   )
-  (symbol (lib_id "Jumper:SolderJumper_2_Open") (at 60.452 230.124 0) (unit 1)
+  (symbol (lib_id "KNeoPix.symbols:SolderJumper_2_Open") (at 60.452 230.124 0) (unit 1)
     (in_bom yes) (on_board yes) (dnp no)
     (property "Reference" "JP3" (at 57.404 224.79 0)
@@
     )
   )
-  (symbol (lib_id "Device:C") (at 43.18 85.852 0) (unit 1)
+  (symbol (lib_id "KNeoPix.symbols:C") (at 43.18 85.852 0) (unit 1)
     (in_bom yes) (on_board yes) (dnp no)
     (property "Reference" "C2" (at 39.37 83.312 0)
@@
     )
   )
-  (symbol (lib_id "Connector_Generic:Conn_01x05") (at 270.51 123.698 0) (unit 1)
+  (symbol (lib_id "KNeoPix.symbols:Conn_01x05") (at 270.51 123.698 0) (unit 1)
     (in_bom yes) (on_board yes) (dnp no)
     (property "Reference" "J6" (at 272.542 123.063 0)
@@
     )
   )
-  (symbol (lib_id "Device:C") (at 273.812 187.706 0) (unit 1)
+  (symbol (lib_id "KNeoPix.symbols:C") (at 273.812 187.706 0) (unit 1)
     (in_bom yes) (on_board yes) (dnp no)
     (property "Reference" "C7" (at 278.892 187.706 0)
@@
     )
   )
-  (symbol (lib_id "Jumper:SolderJumper_2_Open") (at 80.772 140.716 90) (unit 1)
+  (symbol (lib_id "KNeoPix.symbols:SolderJumper_2_Open") (at 80.772 140.716 90) (unit 1)
     (in_bom yes) (on_board yes) (dnp no)
     (property "Reference" "JP6" (at 80.772 128.524 90)
