File: OpenKNXiaO-Mini.kicad_pcb (KiCad board)
At the start: 2 copper layers, 23 x 27 mm, 11 parts, among them J1 Conn_KNX, J2 Conn_01x05, J3 Conn_01x12, SW1 Prog BTN, U1 Seeeduino XIAO

Commit message: Fixed Logo & Version rendering and enabled knx bcu description on back site
Changed lines of the file:
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@@
     (pcbplotparams
       (layerselection 0x0000030_7ffffffe)
-      (plot_on_all_layers_selection 0x0001000_00000000)
+      (plot_on_all_layers_selection 0x0001030_00000000)
       (disableapertmacros false)
       (usegerberextensions false)
@@
       (outputformat 3)
       (mirror false)
-      (drillshape 0)
+      (drillshape 2)
       (scaleselection 1)
       (outputdirectory "DXF")
@@
         (effects (font (size 1 1) (thickness 0.15)))
     )
-    (fp_line (start -4.06 -1.4777) (end 3.27 -1.48)
+    (fp_line (start -4.065 -1.47885) (end 3.265 -1.48115)
       (stroke (width 0.1) (type default)) (layer "F.SilkS"))
     (fp_line (start -4.06 1.92) (end -4.06 -1.4777)
@@
     (fp_line (start 3.27 1.92) (end -4.06 1.92)
       (stroke (width 0.1) (type default)) (layer "F.SilkS"))
-    (pad "" smd rect (at -0.42 0.22 90) (size 7.38 3.4) (layers "F.SilkS"))
+    (pad "" smd rect (at -0.42 0.22 90) (size 7.38 3.4) (layers "Eco1.User"))
   )
   (footprint "KNeoPix:SolderJumper-2_P1.3mm_Open_Pad1.0x1.5mm" (layer "F.Cu")
@@
     (property "ki_keywords" "solder jumper SPST")
     (attr exclude_from_pos_files)
-    (fp_text reference "JP1" (at 2.25 -0.17) (layer "F.SilkS")
+    (fp_text reference "JP1" (at -1.83 0 90) (layer "F.SilkS")
         (effects (font (size 0.5 0.5) (thickness 0.125)))
     )
     (fp_text value "KNX Pin SAVE - Optional" (at 0.24 0.98) (layer "F.SilkS") hide
+        (effects (font (size 0.5 0.5) (thickness 0.125)))
+    )
+    (fp_text user "D10" (at 2.19 -0.03 unlocked) (layer "F.SilkS")
         (effects (font (size 0.5 0.5) (thickness 0.125)))
     )
@@
     (property "ki_keywords" "cap capacitor")
     (attr smd)
-    (fp_text reference "C1" (at 1.84 -0.27 180) (layer "F.SilkS")
+    (fp_text reference "C1" (at 0 0 180) (layer "F.SilkS")
         (effects (font (size 0.5 0.5) (thickness 0.125)))
     )
@@
         (effects (font (size 1 1) (thickness 0.15)))
     )
-    (fp_text user "SAVE" (at -1.16 5.075 90 unlocked) (layer "B.SilkS") hide
+    (fp_text user "SAVE" (at -1.19 5.075 90 unlocked) (layer "B.SilkS")
         (effects (font (size 0.5 0.5) (thickness 0.125)) (justify mirror))
     )
-    (fp_text user "KNX+" (at -1.16 0 90 unlocked) (layer "B.SilkS") hide
+    (fp_text user "KNX+" (at -1.2 0 90 unlocked) (layer "B.SilkS")
         (effects (font (size 0.5 0.5) (thickness 0.125)) (justify mirror))
     )
-    (fp_text user "3V3" (at -1.16 12.65 90 unlocked) (layer "B.SilkS") hide
+    (fp_text user "3V3" (at -1.17 12.68 90 unlocked) (layer "B.SilkS")
         (effects (font (size 0.5 0.5) (thickness 0.125)) (justify mirror))
     )
-    (fp_text user "KNX-" (at -1.16 2.525 90 unlocked) (layer "B.SilkS") hide
+    (fp_text user "KNX-" (at -1.2 2.525 90 unlocked) (layer "B.SilkS")
         (effects (font (size 0.5 0.5) (thickness 0.125)) (justify mirror))
     )
-    (fp_text user "TX" (at -1.16 10.15 90 unlocked) (layer "B.SilkS") hide
+    (fp_text user "TX" (at -1.18 10.15 90 unlocked) (layer "B.SilkS")
         (effects (font (size 0.5 0.5) (thickness 0.125)) (justify mirror))
     )
-    (fp_text user "5V" (at -1.16 15.25 90 unlocked) (layer "B.SilkS") hide
+    (fp_text user "5V" (at -1.17 15.25 90 unlocked) (layer "B.SilkS")
         (effects (font (size 0.5 0.5) (thickness 0.125)) (justify mirror))
     )
-    (fp_text user "RX" (at -1.16 7.6 90 unlocked) (layer "B.SilkS") hide
+    (fp_text user "RX" (at -1.18 7.6 90 unlocked) (layer "B.SilkS")
         (effects (font (size 0.5 0.5) (thickness 0.125)) (justify mirror))
     )
