File: OpenKNXiaO-Mini.kicad_pcb (KiCad board)
At the start: 2 copper layers, 23 x 27 mm, 11 parts, among them J1 Conn_KNX, J2 Conn_01x05, J3 Conn_01x12, SW1 Prog BTN, U1 Seeeduino XIAO

Commit message: last circuit check
Routing:
- net KNX_GND: track 80.7 -> 81.7 mm
- net D8: track 17.3 -> 18.0 mm
- net D5_SCL: track 17.6 -> 18.3 mm
- net S_3V3: track 31.9 -> 32.5 mm
- net D10: track 31.9 -> 32.5 mm
